Commit message: fix: uppercase leg link names + drop _Link suffix to match Thunder asset regex

File: urdf/wheeled_legged_dog_v3.urdf (robot description, URDF)
Before this commit: robot wheeled_legged_dog_v3, 21 links, 20 joints
Links:
- removed link fl_calf_Link
- removed link fl_foot_Link
- removed link fl_hip_Link
- removed link fl_thigh_Link
- removed link fr_calf_Link
- removed link fr_foot_Link
- removed link fr_hip_Link
- removed link fr_thigh_Link
- removed link rl_calf_Link
- removed link rl_foot_Link
- removed link rl_hip_Link
- removed link rl_thigh_Link
- removed link rr_calf_Link
- removed link rr_foot_Link
- removed link rr_hip_Link
- removed link rr_thigh_Link
- added link FL_calf, mass 1.89384; collision box size=0.18 0.04 0.045; collision cylinder length=0.03 radius=0.0635
- added link FL_foot, mass 0.32377; collision cylinder length=0.05617 radius=0.12; visual mesh filename=../meshes/fl_foot_Link.STL
- added link FL_hip, mass 1.78126; collision cylinder length=0.048 radius=0.06; visual mesh filename=../meshes/fl_hip_Link.STL
- added link FL_thigh, mass 2.40982; collision box size=0.18 0.03 0.06; collision cylinder length=0.03 radius=0.064
- added link FR_calf, mass 1.89384; collision box size=0.18 0.04 0.045; collision cylinder length=0.03 radius=0.0635
- added link FR_foot, mass 0.32377; collision cylinder length=0.05617 radius=0.12; visual mesh filename=../meshes/fr_foot_Link.STL
- added link FR_hip, mass 1.78126; collision cylinder length=0.048 radius=0.06; visual mesh filename=../meshes/fr_hip_Link.STL
- added link FR_thigh, mass 2.40982; collision box size=0.18 0.03 0.06; collision cylinder length=0.03 radius=0.064
- added link RL_calf, mass 1.89384; collision box size=0.18 0.04 0.045; collision cylinder length=0.03 radius=0.0635
- added link RL_foot, mass 0.32377; collision cylinder length=0.05617 radius=0.12; visual mesh filename=../meshes/rl_foot_Link.STL
- added link RL_hip, mass 1.78126; collision cylinder length=0.048 radius=0.06; visual mesh filename=../meshes/rl_hip_Link.STL
- added link RL_thigh, mass 2.40982; collision box size=0.18 0.03 0.06; collision cylinder length=0.03 radius=0.064
- added link RR_calf, mass 1.89384; collision box size=0.18 0.04 0.045; collision cylinder length=0.03 radius=0.0635
- added link RR_foot, mass 0.32377; collision cylinder length=0.05617 radius=0.12; visual mesh filename=../meshes/rr_foot_Link.STL
- added link RR_hip, mass 1.78126; collision cylinder length=0.048 radius=0.06; visual mesh filename=../meshes/rr_hip_Link.STL
- added link RR_thigh, mass 2.40982; collision box size=0.18 0.03 0.06; collision cylinder length=0.03 radius=0.064
Joints:
- joint fl_calf_joint: child fl_calf_Link -> FL_calf; parent fl_thigh_Link -> FL_thigh
- joint fl_foot_joint: child fl_foot_Link -> FL_foot; parent fl_calf_Link -> FL_calf
- joint fl_hip_joint: child fl_hip_Link -> FL_hip
- joint fl_thigh_joint: child fl_thigh_Link -> FL_thigh; parent fl_hip_Link -> FL_hip
- joint fr_calf_joint: child fr_calf_Link -> FR_calf; parent fr_thigh_Link -> FR_thigh
- joint fr_foot_joint: child fr_foot_Link -> FR_foot; parent fr_calf_Link -> FR_calf
- joint fr_hip_joint: child fr_hip_Link -> FR_hip
- joint fr_thigh_joint: child fr_thigh_Link -> FR_thigh; parent fr_hip_Link -> FR_hip
- joint rl_calf_joint: child rl_calf_Link -> RL_calf; parent rl_thigh_Link -> RL_thigh
- joint rl_foot_joint: child rl_foot_Link -> RL_foot; parent rl_calf_Link -> RL_calf
- joint rl_hip_joint: child rl_hip_Link -> RL_hip
- joint rl_thigh_joint: child rl_thigh_Link -> RL_thigh; parent rl_hip_Link -> RL_hip
- joint rr_calf_joint: child rr_calf_Link -> RR_calf; parent rr_thigh_Link -> RR_thigh
- joint rr_foot_joint: child rr_foot_Link -> RR_foot; parent rr_calf_Link -> RR_calf
- joint rr_hip_joint: child rr_hip_Link -> RR_hip
- joint rr_thigh_joint: child rr_thigh_Link -> RR_thigh; parent rr_hip_Link -> RR_hip

Commit message: Align Thunder v3 URDF joints with RobotLab naming
The RobotLab Thunder and Hist tasks expect uppercase leg-prefix joint names, so the asset URDF now exports the same FR/FL/RR/RL motion joints while leaving link names and sensor fixed joints unchanged.

Constraint: RobotLab Hist/Thunder configs use uppercase joint selectors

Confidence: high

Scope-risk: narrow

Tested: Parsed URDF XML; verified 21 links, 20 joints, base_link root, 21 unique mesh refs present, uppercase motion joint set complete

Not-tested: Isaac URDF import from this GitHub clone

File: urdf/wheeled_legged_dog_v3.urdf (robot description, URDF)
Before this commit: robot wheeled_legged_dog_v3, 21 links, 20 joints
Joints:
- removed joint fl_calf_joint
- removed joint fl_foot_joint
- removed joint fl_hip_joint
- removed joint fl_thigh_joint
- removed joint fr_calf_joint
- removed joint fr_foot_joint
- removed joint fr_hip_joint
- removed joint fr_thigh_joint
- removed joint rl_calf_joint
- removed joint rl_foot_joint
- removed joint rl_hip_joint
- removed joint rl_thigh_joint
- removed joint rr_calf_joint
- removed joint rr_foot_joint
- removed joint rr_hip_joint
- removed joint rr_thigh_joint
- added joint FL_calf_joint: type revolute, parent FL_thigh, child FL_calf, origin xyz=-0.24954 0.057 -0.01515 rpy=0 0 0, axis 0 -1 0, limit lower=-3.14 upper=0 effort=0 velocity=0
- added joint FL_foot_joint: type continuous, parent FL_calf, child FL_foot, origin xyz=0.24443 0.061 0.0525 rpy=0 0 0, axis 0 -1 0, limit lower=0 upper=0 effort=0 velocity=0
- added joint FL_hip_joint: type revolute, parent base_link, child FL_hip, origin xyz=0.2395 0.065 0.08065 rpy=0 0 0, axis -1 0 0, limit lower=-0.41 upper=0.41 effort=0 velocity=0
- added joint FL_thigh_joint: type revolute, parent FL_hip, child FL_thigh, origin xyz=0.078 0.0795 0 rpy=0 0 0, axis 0 -1 0, limit lower=0 upper=3.14 effort=0 velocity=0
- added joint FR_calf_joint: type revolute, parent FR_thigh, child FR_calf, origin xyz=-0.24954 -0.057 -0.01515 rpy=0 0 0, axis 0 1 0, limit lower=0 upper=3.14 effort=0 velocity=0
- added joint FR_foot_joint: type continuous, parent FR_calf, child FR_foot, origin xyz=0.24443 -0.061 0.0525 rpy=0 0 0, axis 0 1 0, limit lower=0 upper=0 effort=0 velocity=0
- added joint FR_hip_joint: type revolute, parent base_link, child FR_hip, origin xyz=0.2395 -0.065 0.08065 rpy=0 0 0, axis -1 0 0, limit lower=-0.41 upper=0.41 effort=0 velocity=0
- added joint FR_thigh_joint: type revolute, parent FR_hip, child FR_thigh, origin xyz=0.078 -0.0795 0 rpy=0 0 0, axis 0 1 0, limit lower=-3.14 upper=0 effort=0 velocity=0
- added joint RL_calf_joint: type revolute, parent RL_thigh, child RL_calf, origin xyz=0.24954 0.057 -0.01515 rpy=0 0 0, axis 0 -1 0, limit lower=0 upper=6.28 effort=0 velocity=0
- added joint RL_foot_joint: type continuous, parent RL_calf, child RL_foot, origin xyz=-0.24443 0.061 0.0525 rpy=0 0 0, axis 0 -1 0, limit lower=0 upper=0 effort=0 velocity=0
- added joint RL_hip_joint: type revolute, parent base_link, child RL_hip, origin xyz=-0.2395 0.065 0.08065 rpy=0 0 0, axis 1 0 0, limit lower=-0.41 upper=0.41 effort=0 velocity=0
- added joint RL_thigh_joint: type revolute, parent RL_hip, child RL_thigh, origin xyz=-0.078 0.0795 0 rpy=0 0 0, axis 0 -1 0, limit lower=-3.14 upper=0 effort=0 velocity=0
- added joint RR_calf_joint: type revolute, parent RR_thigh, child RR_calf, origin xyz=0.24954 -0.057 -0.01515 rpy=0 0 0, axis 0 1 0, limit lower=-6.28 upper=0 effort=0 velocity=0
- added joint RR_foot_joint: type continuous, parent RR_calf, child RR_foot, origin xyz=-0.24443 -0.061 0.0525 rpy=0 0 0, axis 0 1 0, limit lower=0 upper=0 effort=0 velocity=0
- added joint RR_hip_joint: type revolute, parent base_link, child RR_hip, origin xyz=-0.2395 -0.065 0.08065 rpy=0 0 0, axis 1 0 0, limit lower=-0.41 upper=0.41 effort=0 velocity=0
- added joint RR_thigh_joint: type revolute, parent RR_hip, child RR_thigh, origin xyz=-0.078 -0.0795 0 rpy=0 0 0, axis 0 1 0, limit lower=0 upper=3.14 effort=0 velocity=0
