Commit message: Stabilize Thunder v3 dynamics around corrected CAD inertials
The May 2 CAD export fixes the wheel assembly mass and the calf/thigh inertial alignment, but it is not safe as a direct training URDF because its exported names and joint metadata do not match RobotLab expectations. The primary asset therefore keeps the RobotLab-compatible structure and imports only the corrected inertial blocks.

Constraint: RobotLab configs depend on canonical link/joint names and continuous wheel joints

Rejected: Replace the primary URDF with the raw CAD export | it uses lowercase _Link names, package mesh paths, zero effort/velocity metadata, and wheel limit tags

Confidence: high

Scope-risk: moderate

Directive: Do not copy raw CAD joint limits or effort fields into the primary training asset without RobotLab import and wheel-drive checks

Tested: Parsed primary URDF, XML copy, and raw CAD archive; verified URDF/XML byte sync, 21 links, 20 joints, 48.79163 kg total mass, wheel axes, continuous wheel joints, and leg effort/velocity metadata

Not-tested: Isaac Lab runtime import after this push

File: urdf/legacy/thunder_v3_cad_2026-05-02.urdf (robot description, URDF)
Before this commit: robot thunder_v3, 21 links, 20 joints
Links:
- removed link FL_calf
- removed link FL_foot
- removed link FL_hip
- removed link FL_thigh
- removed link FR_calf
- removed link FR_foot
- removed link FR_hip
- removed link FR_thigh
- removed link RL_calf
- removed link RL_foot
- removed link RL_hip
- removed link RL_thigh
- removed link RR_calf
- removed link RR_foot
- removed link RR_hip
- removed link RR_thigh
- added link fl_calf_Link, mass 1.89384; collision box size=0.18 0.04 0.045; collision cylinder length=0.03 radius=0.0635
- added link fl_foot_Link, mass 1.40377; collision cylinder length=0.05617 radius=0.12; visual mesh filename=package://轮足狗机器人v3/meshes/fl_foot_Link.STL
- added link fl_hip_Link, mass 1.78126; collision cylinder length=0.048 radius=0.06; visual mesh filename=package://轮足狗机器人v3/meshes/fl_hip_Link.STL
- added link fl_thigh_Link, mass 2.40982; collision box size=0.18 0.03 0.06; collision cylinder length=0.03 radius=0.064
- added link fr_calf_Link, mass 1.89384; collision box size=0.18 0.04 0.045; collision cylinder length=0.03 radius=0.0635
- added link fr_foot_Link, mass 1.40377; collision cylinder length=0.05617 radius=0.12; visual mesh filename=package://轮足狗机器人v3/meshes/fr_foot_Link.STL
- added link fr_hip_Link, mass 1.78126; collision cylinder length=0.048 radius=0.06; visual mesh filename=package://轮足狗机器人v3/meshes/fr_hip_Link.STL
- added link fr_thigh_Link, mass 2.40982; collision box size=0.18 0.03 0.06; collision cylinder length=0.03 radius=0.064
- added link rl_calf_Link, mass 1.89384; collision box size=0.18 0.04 0.045; collision cylinder length=0.03 radius=0.0635
- added link rl_foot_Link, mass 1.40377; collision cylinder length=0.05617 radius=0.12; visual mesh filename=package://轮足狗机器人v3/meshes/rl_foot_Link.STL
- added link rl_hip_Link, mass 1.78126; collision cylinder length=0.048 radius=0.06; visual mesh filename=package://轮足狗机器人v3/meshes/rl_hip_Link.STL
- added link rl_thigh_Link, mass 2.40982; collision box size=0.18 0.03 0.06; collision cylinder length=0.03 radius=0.064
- added link rr_calf_Link, mass 1.89384; collision box size=0.18 0.04 0.045; collision cylinder length=0.03 radius=0.0635
- added link rr_foot_Link, mass 1.40377; collision cylinder length=0.05617 radius=0.12; visual mesh filename=package://轮足狗机器人v3/meshes/rr_foot_Link.STL
- added link rr_hip_Link, mass 1.78126; collision cylinder length=0.048 radius=0.06; visual mesh filename=package://轮足狗机器人v3/meshes/rr_hip_Link.STL
- added link rr_thigh_Link, mass 2.40982; collision box size=0.18 0.03 0.06; collision cylinder length=0.03 radius=0.064
- link base_link: geometry collision box size=0.05 0.27 0.14; collision box size=0.05 0.27 0.14
- link camera1_Link: geometry visual mesh filename=package://轮足狗机器人v3/meshes/camera1_Link.STL
- link camera2_Link: geometry visual mesh filename=package://轮足狗机器人v3/meshes/camera2_Link.STL
- link lidar1_Link: geometry visual mesh filename=package://轮足狗机器人v3/meshes/lidar1_Link.STL
- link lidar2_Link: geometry collision box size=0.0768 0.0768 0.0801; visual mesh filename=package://轮足狗机器人v3/meshes/lidar2_Link.STL
Joints:
- removed joint FL_calf_joint
- removed joint FL_foot_joint
- removed joint FL_hip_joint
- removed joint FL_thigh_joint
- removed joint FR_calf_joint
- removed joint FR_foot_joint
- removed joint FR_hip_joint
- removed joint FR_thigh_joint
- removed joint RL_calf_joint
- removed joint RL_foot_joint
- removed joint RL_hip_joint
- removed joint RL_thigh_joint
- removed joint RR_calf_joint
- removed joint RR_foot_joint
- removed joint RR_hip_joint
- removed joint RR_thigh_joint
- added joint fl_calf_joint: type revolute, parent fl_thigh_Link, child fl_calf_Link, origin xyz=-0.24954 0.057 -0.01515 rpy=0 0 0, axis 0 -1 0, limit lower=-3.14 upper=0 effort=0 velocity=0
- added joint fl_foot_joint: type continuous, parent fl_calf_Link, child fl_foot_Link, origin xyz=0.24443 0.061 0.0525 rpy=0 0 0, axis 0 -1 0, limit effort=0 velocity=0
- added joint fl_hip_joint: type revolute, parent base_link, child fl_hip_Link, origin xyz=0.2395 0.065 0.08065 rpy=0 0 0, axis -1 0 0, limit lower=-0.41 upper=0.41 effort=0 velocity=0
- added joint fl_thigh_joint: type revolute, parent fl_hip_Link, child fl_thigh_Link, origin xyz=0.078 0.0795 0 rpy=0 0 0, axis 0 -1 0, limit lower=0 upper=3.14 effort=0 velocity=0
- added joint fr_calf_joint: type revolute, parent fr_thigh_Link, child fr_calf_Link, origin xyz=-0.24954 -0.057 -0.01515 rpy=0 0 0, axis 0 1 0, limit lower=0 upper=3.14 effort=0 velocity=0
- added joint fr_foot_joint: type continuous, parent fr_calf_Link, child fr_foot_Link, origin xyz=0.24443 -0.061 0.0525 rpy=0 0 0, axis 0 1 0, limit effort=0 velocity=0
- added joint fr_hip_joint: type revolute, parent base_link, child fr_hip_Link, origin xyz=0.2395 -0.065 0.08065 rpy=0 0 0, axis -1 0 0, limit lower=-0.41 upper=0.41 effort=0 velocity=0
- added joint fr_thigh_joint: type revolute, parent fr_hip_Link, child fr_thigh_Link, origin xyz=0.078 -0.0795 0 rpy=0 0 0, axis 0 1 0, limit lower=-3.14 upper=0 effort=0 velocity=0
- added joint rl_calf_joint: type revolute, parent rl_thigh_Link, child rl_calf_Link, origin xyz=0.24954 0.057 -0.01515 rpy=0 0 0, axis 0 -1 0, limit lower=0 upper=6.28 effort=0 velocity=0
- added joint rl_foot_joint: type continuous, parent rl_calf_Link, child rl_foot_Link, origin xyz=-0.24443 0.061 0.0525 rpy=0 0 0, axis 0 -1 0, limit effort=0 velocity=0
- added joint rl_hip_joint: type revolute, parent base_link, child rl_hip_Link, origin xyz=-0.2395 0.065 0.08065 rpy=0 0 0, axis 1 0 0, limit lower=-0.41 upper=0.41 effort=0 velocity=0
- added joint rl_thigh_joint: type revolute, parent rl_hip_Link, child rl_thigh_Link, origin xyz=-0.078 0.0795 0 rpy=0 0 0, axis 0 -1 0, limit lower=-3.14 upper=0 effort=0 velocity=0
- added joint rr_calf_joint: type revolute, parent rr_thigh_Link, child rr_calf_Link, origin xyz=0.24954 -0.057 -0.01515 rpy=0 0 0, axis 0 1 0, limit lower=-6.28 upper=0 effort=0 velocity=0
- added joint rr_foot_joint: type continuous, parent rr_calf_Link, child rr_foot_Link, origin xyz=-0.24443 -0.061 0.0525 rpy=0 0 0, axis 0 1 0, limit effort=0 velocity=0
- added joint rr_hip_joint: type revolute, parent base_link, child rr_hip_Link, origin xyz=-0.2395 -0.065 0.08065 rpy=0 0 0, axis 1 0 0, limit lower=-0.41 upper=0.41 effort=0 velocity=0
- added joint rr_thigh_joint: type revolute, parent rr_hip_Link, child rr_thigh_Link, origin xyz=-0.078 -0.0795 0 rpy=0 0 0, axis 0 1 0, limit lower=0 upper=3.14 effort=0 velocity=0
