Commit message: Make Thunder V4 URDF limits usable
Constraint: V4 assets must remain publishable without renaming package paths or generated mesh references.

Rejected: Renaming all V4 joints to V3-style uppercase | joint-name compatibility is a broader integration contract change.

Confidence: high

Scope-risk: narrow

Directive: Revisit effort and velocity once hardware motor specs are available; current values mirror V3 defaults.

Tested: Parsed thunder_v4 URDF; verified 21 links and 20 joints, no missing graph refs, no missing mesh refs, no zero effort or velocity limits, rear calf limits [-3.14, 3.14], and README has no lowercase v3/v4 display text.

Not-tested: ROS, RobotLab, Isaac Lab, or MuJoCo import/runtime.

Co-authored-by: OmX <omx@oh-my-codex.dev>

File: thunder_v4/urdf/thunder_v4.urdf (robot description, URDF)
Before this commit: robot thunder_v4, 21 links, 20 joints
Joints:
- joint fl_calf_joint: limit lower=-3.14 upper=0 effort=0 velocity=0 -> lower=-3.14 upper=0 effort=120 velocity=17.48
- joint fl_foot_joint: limit effort=0 velocity=0 -> effort=120 velocity=17.48
- joint fl_hip_joint: limit lower=-0.41 upper=0.41 effort=0 velocity=0 -> lower=-0.41 upper=0.41 effort=120 velocity=17.48
- joint fl_thigh_joint: limit lower=0 upper=3.14 effort=0 velocity=0 -> lower=0 upper=3.14 effort=120 velocity=17.48
- joint fr_calf_joint: limit lower=0 upper=3.14 effort=0 velocity=0 -> lower=0 upper=3.14 effort=120 velocity=17.48
- joint fr_foot_joint: limit effort=0 velocity=0 -> effort=120 velocity=17.48
- joint fr_hip_joint: limit lower=-0.41 upper=0.41 effort=0 velocity=0 -> lower=-0.41 upper=0.41 effort=120 velocity=17.48
- joint fr_thigh_joint: limit lower=-3.14 upper=0 effort=0 velocity=0 -> lower=-3.14 upper=0 effort=120 velocity=17.48
- joint rl_calf_joint: limit lower=0 upper=6.28 effort=0 velocity=0 -> lower=-3.14 upper=3.14 effort=120 velocity=17.48
- joint rl_foot_joint: limit effort=0 velocity=0 -> effort=120 velocity=17.48
- joint rl_hip_joint: limit lower=-0.41 upper=0.41 effort=0 velocity=0 -> lower=-0.41 upper=0.41 effort=120 velocity=17.48
- joint rl_thigh_joint: limit lower=-3.14 upper=0 effort=0 velocity=0 -> lower=-3.14 upper=0 effort=120 velocity=17.48
- joint rr_calf_joint: limit lower=-6.28 upper=0 effort=0 velocity=0 -> lower=-3.14 upper=3.14 effort=120 velocity=17.48
- joint rr_foot_joint: limit effort=0 velocity=0 -> effort=120 velocity=17.48
- joint rr_hip_joint: limit lower=-0.41 upper=0.41 effort=0 velocity=0 -> lower=-0.41 upper=0.41 effort=120 velocity=17.48
- joint rr_thigh_joint: limit lower=0 upper=3.14 effort=0 velocity=0 -> lower=0 upper=3.14 effort=120 velocity=17.48

Commit message: Separate Thunder V4 foot motor limits
Constraint: V4 wheel-foot hardware is documented as the RS02 small-wheel variant.

Rejected: Keeping foot joints on the leg actuator 120 Nm placeholder | the wheel motor has a separate torque and speed envelope.

Confidence: medium

Scope-risk: narrow

Directive: Re-check these values against the exact purchased RS02 revision before sim-to-real tuning.

Tested: Parsed Thunder V4 URDF; verified 21 links and 20 joints, no missing graph or mesh refs, no zero effort or velocity limits, hip/thigh/calf limits stay 120/17.48, and all four foot joints plus CSV metadata use effort 17 and velocity 44.

Not-tested: ROS, RobotLab, Isaac Lab, MuJoCo import, or hardware motor validation.

Co-authored-by: OmX <omx@oh-my-codex.dev>

File: thunder_v4/urdf/thunder_v4.urdf (robot description, URDF)
Before this commit: robot thunder_v4, 21 links, 20 joints
Joints:
- joint fl_foot_joint: limit effort=120 velocity=17.48 -> effort=17 velocity=44
- joint fr_foot_joint: limit effort=120 velocity=17.48 -> effort=17 velocity=44
- joint rl_foot_joint: limit effort=120 velocity=17.48 -> effort=17 velocity=44
- joint rr_foot_joint: limit effort=120 velocity=17.48 -> effort=17 velocity=44
