Commit message: fix: set Thunder V4 wheel collision radius to 95mm

File: thunder_v4/urdf/thunder_v4.urdf (robot description, URDF)
Before this commit: robot thunder_v4, 21 links, 20 joints
Links:
- link fl_foot_Link: geometry collision cylinder length=0.05117 radius=0.095; visual mesh filename=../meshes/fl_foot_Link.STL
- link fr_foot_Link: geometry collision cylinder length=0.05117 radius=0.095; visual mesh filename=../meshes/fr_foot_Link.STL
- link rl_foot_Link: geometry collision cylinder length=0.05117 radius=0.095; visual mesh filename=../meshes/rl_foot_Link.STL
- link rr_foot_Link: geometry collision cylinder length=0.05117 radius=0.095; visual mesh filename=../meshes/rr_foot_Link.STL
